File: eagle/ctrl_encoder.brd (EAGLE design)
At the start: 25.5 x 25.5 mm, 15 parts, among them J1 PAD+SQUARE-1.5X1.5, J10 PAD+SQUARE-1.5X1.5, J11 PAD+SQUARE-1.5X1.5, J2 PAD+SQUARE-1.5X1.5, J3 PAD+SQUARE-1.5X1.5, J4 PAD+SQUARE-1.5X1.5, J5 PAD+SQUARE-1.5X1.5, J6 PAD+SQUARE-1.5X1.5, J7 PAD+SQUARE-1.5X1.5, J8 PAD+SQUARE-1.5X1.5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

Commit message: small changes
Parts:
- removed J8: PAD+SQUARE-1.5X1.5, LockBox:PAD-1.5X1.5
Connections:
- removed net N$10: J8.PAD, U$1.10
- net N$1: now also U$1.10
Routing:
- net N$10: track 37.5 -> 0.00 mm
- net N$1: track 5.64 -> 15.9 mm
Changed lines of the file:
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@@
 <element name="J6" library="LockBox" package="PAD-1.5X1.5" value="PAD+SQUARE-1.5X1.5" x="1.94" y="15.82"/>
 <element name="J7" library="LockBox" package="PAD-1.5X1.5" value="PAD+SQUARE-1.5X1.5" x="1.93" y="18.72"/>
-<element name="J8" library="LockBox" package="PAD-1.5X1.5" value="PAD+SQUARE-1.5X1.5" x="1.92" y="21.52"/>
 <element name="J9" library="LockBox" package="PAD-1.5X1.5" value="PAD+SQUARE-1.5X1.5" x="22.46" y="15.33"/>
 <element name="J10" library="LockBox" package="PAD-1.5X1.5" value="PAD+SQUARE-1.5X1.5" x="22.4" y="13.23"/>
@@
 <wire x1="14.39" y1="17.81" x2="14.01" y2="17.33" width="0.4064" layer="1"/>
 <wire x1="14.01" y1="17.33" x2="14.0284" y2="17.33" width="0.4064" layer="1"/>
-<wire x1="14.0284" y1="17.33" x2="16.1534" y2="15.205" width="0.4064" layer="1"/>
+<wire x1="14.0284" y1="17.33" x2="15.6792" y2="15.6792" width="0.4064" layer="1"/>
+<contactref element="U$1" pad="10"/>
+<wire x1="15.6792" y1="15.6792" x2="16.1534" y2="15.205" width="0.4064" layer="1"/>
+<wire x1="16.1534" y1="7.585" x2="15.115" y2="7.585" width="0.4064" layer="1"/>
+<wire x1="15.115" y1="7.585" x2="14.2" y2="8.5" width="0.4064" layer="1"/>
+<wire x1="14.2" y1="8.5" x2="14.2" y2="14.5" width="0.4064" layer="1"/>
+<wire x1="14.2" y1="14.5" x2="14.7" y2="15" width="0.4064" layer="1"/>
+<wire x1="14.7" y1="15" x2="14.8" y2="15" width="0.4064" layer="1"/>
+<wire x1="14.8" y1="15" x2="15.1" y2="15.3" width="0.4064" layer="1"/>
+<wire x1="15.1" y1="15.3" x2="15.3" y2="15.3" width="0.4064" layer="1"/>
+<wire x1="15.3" y1="15.3" x2="15.6792" y2="15.6792" width="0.4064" layer="1"/>
 </signal>
 <signal name="N$3">
@@
 <wire x1="2.01" y1="18.8" x2="1.93" y2="18.72" width="0.4064" layer="1"/>
 </signal>
-<signal name="N$10">
-<contactref element="U$1" pad="10"/>
-<contactref element="J8" pad="PAD"/>
-<wire x1="16.1534" y1="7.585" x2="18.085" y2="7.585" width="0.4064" layer="1"/>
-<wire x1="18.085" y1="7.585" x2="20.6" y2="10.1" width="0.4064" layer="1"/>
-<wire x1="20.6" y1="10.1" x2="20.6" y2="21.6" width="0.4064" layer="1"/>
-<wire x1="20.6" y1="21.6" x2="18.4" y2="23.8" width="0.4064" layer="1"/>
-<wire x1="18.4" y1="23.8" x2="6.3" y2="23.8" width="0.4064" layer="1"/>
-<wire x1="6.3" y1="23.8" x2="4" y2="21.5" width="0.4064" layer="1"/>
-<wire x1="4" y1="21.5" x2="1.94" y2="21.5" width="0.4064" layer="1"/>
-<wire x1="1.94" y1="21.5" x2="1.92" y2="21.52" width="0.4064" layer="1"/>
-</signal>
 <signal name="GND">
