File: eagle/ctrl_encoder.sch (EAGLE design)
At the start: 15 parts, among them J1 PAD+SQUARE-1.5X1.5, J10 PAD+SQUARE-1.5X1.5, J11 PAD+SQUARE-1.5X1.5, J2 PAD+SQUARE-1.5X1.5, J3 PAD+SQUARE-1.5X1.5, J4 PAD+SQUARE-1.5X1.5, J5 PAD+SQUARE-1.5X1.5, J6 PAD+SQUARE-1.5X1.5, J7 PAD+SQUARE-1.5X1.5, J8 PAD+SQUARE-1.5X1.5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

Commit message: small changes
Parts:
- removed J8: PAD+SQUARE-1.5X1.5, LockBox:PAD+SQUARE-1.5X1.5
Connections:
- removed net N$10: J8.PAD, U$1.IN0
- net N$1: now also U$1.IN0
Changed lines of the file:
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@@
 <part name="J6" library="LockBox" deviceset="PAD+SQUARE" device="-1.5X1.5"/>
 <part name="J7" library="LockBox" deviceset="PAD+SQUARE" device="-1.5X1.5"/>
-<part name="J8" library="LockBox" deviceset="PAD+SQUARE" device="-1.5X1.5"/>
 <part name="J9" library="LockBox" deviceset="PAD+SQUARE" device="-1.5X1.5"/>
 <part name="J10" library="LockBox" deviceset="PAD+SQUARE" device="-1.5X1.5"/>
@@
 <instance part="J6" gate="PAD" x="-41.91" y="10.16"/>
 <instance part="J7" gate="PAD" x="-41.91" y="6.35"/>
-<instance part="J8" gate="PAD" x="-41.91" y="2.54"/>
 <instance part="J9" gate="PAD" x="11.43" y="26.67" rot="R180"/>
 <instance part="J10" gate="PAD" x="11.43" y="22.86" rot="R180"/>
@@
 <segment>
 <pinref part="U$1" gate="G$1" pin="VCC"/>
-<wire x1="-13.97" y1="-10.16" x2="-13.97" y2="-19.05" width="0.1524" layer="91"/>
+<wire x1="-13.97" y1="-10.16" x2="-13.97" y2="-13.97" width="0.1524" layer="91"/>
+<wire x1="-13.97" y1="-13.97" x2="-13.97" y2="-19.05" width="0.1524" layer="91"/>
 <wire x1="-13.97" y1="-19.05" x2="-15.24" y2="-20.32" width="0.1524" layer="91"/>
 <pinref part="C1" gate="G$1" pin="2"/>
@@
 <junction x="-15.24" y="-25.4"/>
 <pinref part="VCC" gate="PAD" pin="PAD"/>
+<pinref part="U$1" gate="G$1" pin="IN0"/>
+<wire x1="-29.21" y1="2.54" x2="-26.67" y2="2.54" width="0.1524" layer="91"/>
+<wire x1="-13.97" y1="-13.97" x2="-29.21" y2="-13.97" width="0.1524" layer="91"/>
+<wire x1="-29.21" y1="-13.97" x2="-29.21" y2="2.54" width="0.1524" layer="91"/>
+<junction x="-13.97" y="-13.97"/>
 </segment>
 </net>
@@
 </segment>
 </net>
-<net name="N$10" class="0">
-<segment>
-<pinref part="U$1" gate="G$1" pin="IN0"/>
-<pinref part="J8" gate="PAD" pin="PAD"/>
-<wire x1="-26.67" y1="2.54" x2="-39.37" y2="2.54" width="0.1524" layer="91"/>
-</segment>
-</net>
