File: eagle/encoder/ctrl_encoder.sch (EAGLE design)
At the start: 14 parts, among them J1 PAD+SQUARE-1.5X1.5, J10 PAD+SQUARE-1.5X1.5, J11 PAD+SQUARE-1.5X1.5, J2 PAD+SQUARE-1.5X1.5, J3 PAD+SQUARE-1.5X1.5, J4 PAD+SQUARE-1.5X1.5, J5 PAD+SQUARE-1.5X1.5, J6 PAD+SQUARE-1.5X1.5, J7 PAD+SQUARE-1.5X1.5, J9 PAD+SQUARE-1.5X1.5

Commit message: Replaced surface mount pads with through hole pads.  Added a polygon to the .brd and increased the size of the isolate from 10mil to 20mils, this should prevent solder from bridging to the remaining copper on the test board.  Also increased the spacing of the pads.
Parts:
- GND, J1, J10, J11, J2, J3, J4, J5, J6, J7, J9, VCC: value PAD+SQUARE-1.5X1.5 -> PAD; device LockBox:PAD+SQUARE-1.5X1.5 -> LockBox:PAD
Changed lines of the file:
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@@
 <setting verticaltext="up"/>
 </settings>
-<grid distance="0.05" unitdist="inch" unit="inch" style="lines" multiple="1" display="yes" altdistance="0.01" altunitdist="inch" altunit="inch"/>
+<grid distance="0.5" unitdist="mm" unit="mm" style="lines" multiple="1" display="no" altdistance="0.01" altunitdist="inch" altunit="inch"/>
 <layers>
 <layer number="1" name="Top" color="4" fill="1" visible="no" active="no"/>
@@
 <part name="U$1" library="LockBox" deviceset="SN74HC148" device="DR"/>
 <part name="C1" library="LockBox" deviceset="C" device=""/>
-<part name="J1" library="LockBox" deviceset="PAD+SQUARE" device="-1.5X1.5"/>
-<part name="J2" library="LockBox" deviceset="PAD+SQUARE" device="-1.5X1.5"/>
-<part name="J3" library="LockBox" deviceset="PAD+SQUARE" device="-1.5X1.5"/>
-<part name="J4" library="LockBox" deviceset="PAD+SQUARE" device="-1.5X1.5"/>
-<part name="J5" library="LockBox" deviceset="PAD+SQUARE" device="-1.5X1.5"/>
-<part name="J6" library="LockBox" deviceset="PAD+SQUARE" device="-1.5X1.5"/>
-<part name="J7" library="LockBox" deviceset="PAD+SQUARE" device="-1.5X1.5"/>
-<part name="J9" library="LockBox" deviceset="PAD+SQUARE" device="-1.5X1.5"/>
-<part name="J10" library="LockBox" deviceset="PAD+SQUARE" device="-1.5X1.5"/>
-<part name="J11" library="LockBox" deviceset="PAD+SQUARE" device="-1.5X1.5"/>
-<part name="GND" library="LockBox" deviceset="PAD+SQUARE" device="-1.5X1.5"/>
-<part name="VCC" library="LockBox" deviceset="PAD+SQUARE" device="-1.5X1.5"/>
+<part name="J1" library="LockBox" deviceset="PAD" device=""/>
+<part name="J2" library="LockBox" deviceset="PAD" device=""/>
+<part name="J3" library="LockBox" deviceset="PAD" device=""/>
+<part name="J4" library="LockBox" deviceset="PAD" device=""/>
+<part name="J5" library="LockBox" deviceset="PAD" device=""/>
+<part name="J6" library="LockBox" deviceset="PAD" device=""/>
+<part name="J7" library="LockBox" deviceset="PAD" device=""/>
+<part name="J9" library="LockBox" deviceset="PAD" device=""/>
+<part name="J10" library="LockBox" deviceset="PAD" device=""/>
+<part name="J11" library="LockBox" deviceset="PAD" device=""/>
+<part name="GND" library="LockBox" deviceset="PAD" device=""/>
+<part name="VCC" library="LockBox" deviceset="PAD" device=""/>
 </parts>
 <sheets>
@@
 <instance part="U$1" gate="G$1" x="-20.32" y="10.16"/>
 <instance part="C1" gate="G$1" x="-10.16" y="-25.4" rot="R270"/>
-<instance part="J1" gate="PAD" x="-41.91" y="29.21"/>
-<instance part="J2" gate="PAD" x="-41.91" y="25.4"/>
-<instance part="J3" gate="PAD" x="-41.91" y="21.59"/>
-<instance part="J4" gate="PAD" x="-41.91" y="17.78"/>
-<instance part="J5" gate="PAD" x="-41.91" y="13.97"/>
-<instance part="J6" gate="PAD" x="-41.91" y="10.16"/>
-<instance part="J7" gate="PAD" x="-41.91" y="6.35"/>
-<instance part="J9" gate="PAD" x="11.43" y="26.67" rot="R180"/>
-<instance part="J10" gate="PAD" x="11.43" y="22.86" rot="R180"/>
-<instance part="J11" gate="PAD" x="11.43" y="19.05" rot="R180"/>
-<instance part="GND" gate="PAD" x="-7.62" y="-34.29" rot="R90"/>
-<instance part="VCC" gate="PAD" x="-15.24" y="-34.29" rot="R90"/>
+<instance part="J1" gate="G$1" x="-41.91" y="29.21"/>
+<instance part="J2" gate="G$1" x="-41.91" y="25.4"/>
+<instance part="J3" gate="G$1" x="-41.91" y="21.59"/>
+<instance part="J4" gate="G$1" x="-41.91" y="17.78"/>
+<instance part="J5" gate="G$1" x="-41.91" y="13.97"/>
+<instance part="J6" gate="G$1" x="-41.91" y="10.16"/>
+<instance part="J7" gate="G$1" x="-41.91" y="6.35"/>
+<instance part="J9" gate="G$1" x="11.43" y="26.67" rot="R180"/>
+<instance part="J10" gate="G$1" x="11.43" y="22.86" rot="R180"/>
+<instance part="J11" gate="G$1" x="11.43" y="19.05" rot="R180"/>
+<instance part="GND" gate="G$1" x="-7.62" y="-34.29" rot="R90"/>
+<instance part="VCC" gate="G$1" x="-15.24" y="-34.29" rot="R90"/>
 </instances>
 <busses>
@@
 <wire x1="-15.24" y1="-25.4" x2="-15.24" y2="-31.75" width="0.1524" layer="91"/>
 <junction x="-15.24" y="-25.4"/>
-<pinref part="VCC" gate="PAD" pin="PAD"/>
+<pinref part="VCC" gate="G$1" pin="PAD"/>
 <pinref part="U$1" gate="G$1" pin="IN0"/>
 <wire x1="-29.21" y1="2.54" x2="-26.67" y2="2.54" width="0.1524" layer="91"/>
@@
 <net name="N$3" class="0">
 <segment>
-<pinref part="J1" gate="PAD" pin="PAD"/>
+<pinref part="J1" gate="G$1" pin="PAD"/>
 <pinref part="U$1" gate="G$1" pin="IN7"/>
 <wire x1="-39.37" y1="29.21" x2="-26.67" y2="29.21" width="0.1524" layer="91"/>
@@
 <segment>
 <pinref part="U$1" gate="G$1" pin="IN6"/>
-<pinref part="J2" gate="PAD" pin="PAD"/>
+<pinref part="J2" gate="G$1" pin="PAD"/>
 <wire x1="-26.67" y1="25.4" x2="-39.37" y2="25.4" width="0.1524" layer="91"/>
 </segment>
@@
 <net name="N$5" class="0">
 <segment>
-<pinref part="J3" gate="PAD" pin="PAD"/>
+<pinref part="J3" gate="G$1" pin="PAD"/>
 <pinref part="U$1" gate="G$1" pin="IN5"/>
 <wire x1="-39.37" y1="21.59" x2="-26.67" y2="21.59" width="0.1524" layer="91"/>
@@
 <segment>
 <pinref part="U$1" gate="G$1" pin="IN4"/>
-<pinref part="J4" gate="PAD" pin="PAD"/>
+<pinref part="J4" gate="G$1" pin="PAD"/>
 <wire x1="-26.67" y1="17.78" x2="-39.37" y2="17.78" width="0.1524" layer="91"/>
 </segment>
@@
 <net name="N$7" class="0">
 <segment>
-<pinref part="J5" gate="PAD" pin="PAD"/>
+<pinref part="J5" gate="G$1" pin="PAD"/>
 <pinref part="U$1" gate="G$1" pin="IN3"/>
 <wire x1="-39.37" y1="13.97" x2="-26.67" y2="13.97" width="0.1524" layer="91"/>
@@
 <segment>
 <pinref part="U$1" gate="G$1" pin="IN2"/>
-<pinref part="J6" gate="PAD" pin="PAD"/>
+<pinref part="J6" gate="G$1" pin="PAD"/>
 <wire x1="-26.67" y1="10.16" x2="-39.37" y2="10.16" width="0.1524" layer="91"/>
 </segment>
@@
 <net name="N$9" class="0">
 <segment>
-<pinref part="J7" gate="PAD" pin="PAD"/>
+<pinref part="J7" gate="G$1" pin="PAD"/>
 <pinref part="U$1" gate="G$1" pin="IN1"/>
 <wire x1="-39.37" y1="6.35" x2="-26.67" y2="6.35" width="0.1524" layer="91"/>
@@
 <wire x1="-7.62" y1="-25.4" x2="-7.62" y2="-31.75" width="0.1524" layer="91"/>
 <junction x="-7.62" y="-25.4"/>
-<pinref part="GND" gate="PAD" pin="PAD"/>
+<pinref part="GND" gate="G$1" pin="PAD"/>
 <wire x1="-5.08" y1="-31.75" x2="-7.62" y2="-31.75" width="0.1524" layer="91"/>
 <junction x="-7.62" y="-31.75"/>
@@
 <segment>
 <pinref part="U$1" gate="G$1" pin="A2"/>
-<pinref part="J9" gate="PAD" pin="PAD"/>
+<pinref part="J9" gate="G$1" pin="PAD"/>
 <wire x1="-1.27" y1="26.67" x2="8.89" y2="26.67" width="0.1524" layer="91"/>
 </segment>
@@
 <segment>
 <pinref part="U$1" gate="G$1" pin="A1"/>
-<pinref part="J10" gate="PAD" pin="PAD"/>
+<pinref part="J10" gate="G$1" pin="PAD"/>
 <wire x1="-1.27" y1="22.86" x2="8.89" y2="22.86" width="0.1524" layer="91"/>
 </segment>
@@
 <segment>
 <pinref part="U$1" gate="G$1" pin="A0"/>
-<pinref part="J11" gate="PAD" pin="PAD"/>
+<pinref part="J11" gate="G$1" pin="PAD"/>
 <wire x1="-1.27" y1="19.05" x2="8.89" y2="19.05" width="0.1524" layer="91"/>
 </segment>
