File: eagle/LCD/LCD_board.brd (EAGLE design)
At the start: 100.5 x 81.4 mm, 7 parts, among them CN1 1X4-CLEANBIG

Commit message: layout dimension change
will try to build tomorrow
Parts:
- moved C1 6.38 mm to (47.2, 16.3)
- moved U$1 6.38 mm to (53.6, 49.4)
- moved C2 6.38 mm to (41.2, 25.4)
- moved DATALINES 6.38 mm to (55.9, 6.57)
- moved R1 6.38 mm to (42.6, 6.40)
- moved R2 6.38 mm to (45.1, 6.40)
- moved CN1 6.38 mm to (5.48, 49.5)
Other:
- board size 100.5 x 81.4 mm -> 93.1 x 60.1 mm
